Commit message: Removed adc sampling rate and fixed cmakes

File: net_ft_description/urdf/ati_axia80_ft_sensor.urdf.xacro (robot description, xacro)
@@ -4,5 +4,4 @@
     <xacro:arg name="ip_address" default="192.168.1.1" />
     <xacro:arg name="rdt_sampling_rate" default="500" />
-    <xacro:arg name="adc_sampling_rate" default="976" />
     <!-- Import macros -->
     <xacro:include filename="$(find net_ft_description)/urdf/ati_axia80_ft_sensor_macro.urdf.xacro" />
@@ -12,6 +11,5 @@
       prefix=""
       ip_address="$(arg ip_address)"
-      rdt_sampling_rate="$(arg rdt_sampling_rate)"
-      adc_sampling_rate="$(arg adc_sampling_rate)">
+      rdt_sampling_rate="$(arg rdt_sampling_rate)">
         <origin xyz="0 0 0" rpy="0 0 0" />
     </xacro:ati_axia80_ft_sensor>

File: net_ft_description/urdf/ati_axia80_ft_sensor_macro.urdf.xacro (robot description, xacro)
@@ -6,6 +6,5 @@
     *origin
     ip_address
-    rdt_sampling_rate
-    adc_sampling_rate">
+    rdt_sampling_rate">
     <joint name="${prefix}fts_joint" type="fixed">
       <!-- The parent link must be read from the robot model it is attached to. -->
@@ -44,6 +43,5 @@
       sensor_type="ati_axia"
       ip_address="${ip_address}"
-      rdt_sampling_rate="${rdt_sampling_rate}"
-      adc_sampling_rate="${adc_sampling_rate}" />
+      rdt_sampling_rate="${rdt_sampling_rate}"/>
   </xacro:macro>
 </robot>

File: net_ft_description/urdf/net_ft_sensor.ros2_control.xacro (robot description, xacro)
@@ -1,5 +1,5 @@
 <?xml version="1.0"?>
 <robot xmlns:xacro="http://www.ros.org/wiki/xacro">
-    <xacro:macro name="net_ft_sensor_ros2_control" params="name prefix ip_address sensor_type rdt_sampling_rate:=500 adc_sampling_rate:=976">
+    <xacro:macro name="net_ft_sensor_ros2_control" params="name prefix ip_address sensor_type rdt_sampling_rate:=500">
         <ros2_control name="${name}" type="sensor">
             <hardware>
@@ -8,5 +8,4 @@
                 <param name="ip_address">${ip_address}</param>
                 <param name="rdt_sampling_rate">${rdt_sampling_rate}</param>
-                <param name="adc_sampling_rate">${adc_sampling_rate}</param>
             </hardware>
             <sensor name="${prefix}tcp_fts_sensor">
