Commit message: Tested with ATI AXIA80 and OnRobot HEX-E

File: net_ft_description/urdf/ati_axia80_ft_sensor_macro.urdf.xacro (robot description, xacro)
@@ -40,6 +40,6 @@
     <xacro:include filename="$(find net_ft_description)/urdf/net_ft_sensor.ros2_control.xacro" />
     <xacro:net_ft_sensor_ros2_control
-      name="NetFTHardwareInterface"
-      sensor_type="ati_axia"
+      name="NetFtHardwareInterface"
+      sensor_type="onrobot"
       ip_address="${ip_address}"
       rdt_sampling_rate="${rdt_sampling_rate}"/>

File: net_ft_description/urdf/net_ft_sensor.ros2_control.xacro (robot description, xacro)
@@ -1,13 +1,13 @@
 <?xml version="1.0"?>
 <robot xmlns:xacro="http://www.ros.org/wiki/xacro">
-    <xacro:macro name="net_ft_sensor_ros2_control" params="name prefix ip_address sensor_type rdt_sampling_rate:=500">
+    <xacro:macro name="net_ft_sensor_ros2_control" params="name ip_address sensor_type rdt_sampling_rate">
         <ros2_control name="${name}" type="sensor">
             <hardware>
-                <plugin>net_ft_driver/NetFTHardwareInterface</plugin>
+                <plugin>net_ft_driver/NetFtHardwareInterface</plugin>
                 <param name="sensor_type">${sensor_type}</param>
                 <param name="ip_address">${ip_address}</param>
                 <param name="rdt_sampling_rate">${rdt_sampling_rate}</param>
             </hardware>
-            <sensor name="${prefix}tcp_fts_sensor">
+            <sensor name="tcp_fts_sensor">
               <state_interface name="force.x"/>
               <state_interface name="force.y"/>
