Commit message: Added sensor description and launch file

File: net_ft_description/urdf/net_ft_sensor.ros2_control.xacro (robot description, xacro)
@@ -1,5 +1,5 @@
 <?xml version="1.0"?>
 <robot xmlns:xacro="http://www.ros.org/wiki/xacro">
-    <xacro:macro name="net_ft_sensor_ros2_control" params="name ip_address sensor_type rdt_sampling_rate:=500 adc_sampling_rate:=976">
+    <xacro:macro name="net_ft_sensor_ros2_control" params="name prefix ip_address sensor_type rdt_sampling_rate:=500 adc_sampling_rate:=976">
         <ros2_control name="${name}" type="sensor">
             <hardware>
@@ -10,5 +10,5 @@
                 <param name="adc_sampling_rate">${adc_sampling_rate}</param>
             </hardware>
-            <sensor name="${prefix}net_ft_sensor">
+            <sensor name="${prefix}tcp_fts_sensor">
               <state_interface name="force.x"/>
               <state_interface name="force.y"/>
@@ -18,11 +18,11 @@
               <state_interface name="torque.z"/>
               <param name="frame_id">tool_link</param>
-              <param name="fx_range">100</param>
-              <param name="fy_range">100</param>
-              <param name="fz_range">100</param>
-              <param name="tx_range">15</param>
-              <param name="ty_range">15</param>
-              <param name="tz_range">15</param>
           </sensor>
+          <gpio name="diagnostic">
+            <state_interface name="packet_count"/>
+            <state_interface name="lost_packets"/>
+            <state_interface name="out_of_order_count"/>
+            <state_interface name="status"/>
+          </gpio>
         </ros2_control>
     </xacro:macro>

Commit message: Fixed descriptions

File: net_ft_description/urdf/net_ft_sensor.ros2_control.xacro (robot description, xacro)
@@ -1,5 +1,5 @@
 <?xml version="1.0"?>
 <robot xmlns:xacro="http://www.ros.org/wiki/xacro">
-    <xacro:macro name="net_ft_sensor_ros2_control" params="name ip_address sensor_type rdt_sampling_rate">
+    <xacro:macro name="net_ft_sensor_ros2_control" params="name ip_address sensor_type rdt_sampling_rate internal_filter_rate">
         <ros2_control name="${name}" type="sensor">
             <hardware>
@@ -8,4 +8,5 @@
                 <param name="ip_address">${ip_address}</param>
                 <param name="rdt_sampling_rate">${rdt_sampling_rate}</param>
+                <param name="internal_filter_rate">${internal_filter_rate}</param>
             </hardware>
             <sensor name="tcp_fts_sensor">

File: net_ft_description/urdf/net_ft_sensor.urdf.xacro (robot description, xacro)
@@ -5,4 +5,5 @@
     <xacro:arg name="rdt_sampling_rate" default="500" />
     <xacro:arg name="sensor_type" default="ati_axia80" />
+    <xacro:arg name="internal_filter_rate" default="0" />
     <link name="world" />
     <xacro:include filename="$(find net_ft_description)/urdf/net_ft_sensor_macro.urdf.xacro" />
@@ -12,5 +13,6 @@
       ip_address="$(arg ip_address)"
       rdt_sampling_rate="$(arg rdt_sampling_rate)"
-      sensor_type="$(arg sensor_type)">
+      sensor_type="$(arg sensor_type)"
+      internal_filter_rate="$(arg internal_filter_rate)">
         <origin xyz="0 0 0" rpy="0 0 0" />
     </xacro:net_ft_sensor>

File: net_ft_description/urdf/net_ft_sensor_macro.urdf.xacro (robot description, xacro)
@@ -7,5 +7,6 @@
     ip_address
     rdt_sampling_rate
-    sensor_type">
+    sensor_type
+    internal_filter_rate">
     <xacro:macro name="cylinder_inertial" params="radius length mass *origin">
       <inertial>
@@ -63,5 +64,6 @@
       sensor_type="${sensor_type}"
       ip_address="${ip_address}"
-      rdt_sampling_rate="${rdt_sampling_rate}"/>
+      rdt_sampling_rate="${rdt_sampling_rate}"
+      internal_filter_rate="${internal_filter_rate}"/>
   </xacro:macro>
 </robot>

Commit message: Added sensor zeroing as optional functionality

File: net_ft_description/urdf/net_ft_sensor.ros2_control.xacro (robot description, xacro)
@@ -1,5 +1,5 @@
 <?xml version="1.0"?>
 <robot xmlns:xacro="http://www.ros.org/wiki/xacro">
-    <xacro:macro name="net_ft_sensor_ros2_control" params="name ip_address sensor_type rdt_sampling_rate internal_filter_rate">
+    <xacro:macro name="net_ft_sensor_ros2_control" params="name ip_address sensor_type rdt_sampling_rate internal_filter_rate use_hardware_biasing">
         <ros2_control name="${name}" type="sensor">
             <hardware>
@@ -9,4 +9,5 @@
                 <param name="rdt_sampling_rate">${rdt_sampling_rate}</param>
                 <param name="internal_filter_rate">${internal_filter_rate}</param>
+                <param name="use_hardware_biasing">${use_hardware_biasing}</param>
             </hardware>
             <sensor name="tcp_fts_sensor">

File: net_ft_description/urdf/net_ft_sensor.urdf.xacro (robot description, xacro)
@@ -6,4 +6,5 @@
     <xacro:arg name="sensor_type" default="ati_axia80" />
     <xacro:arg name="internal_filter_rate" default="0" />
+    <xacro:arg name="use_hardware_biasing" default="false" />
     <link name="world" />
     <xacro:include filename="$(find net_ft_description)/urdf/net_ft_sensor_macro.urdf.xacro" />
@@ -14,5 +15,6 @@
       rdt_sampling_rate="$(arg rdt_sampling_rate)"
       sensor_type="$(arg sensor_type)"
-      internal_filter_rate="$(arg internal_filter_rate)">
+      internal_filter_rate="$(arg internal_filter_rate)"
+      use_hardware_biasing="$(use_hardware_biasing)">
         <origin xyz="0 0 0" rpy="0 0 0" />
     </xacro:net_ft_sensor>

File: net_ft_description/urdf/net_ft_sensor_macro.urdf.xacro (robot description, xacro)
@@ -8,5 +8,6 @@
     rdt_sampling_rate
     sensor_type
-    internal_filter_rate">
+    internal_filter_rate
+    use_hardware_biasing">
     <xacro:macro name="cylinder_inertial" params="radius length mass *origin">
       <inertial>
@@ -71,5 +72,6 @@
       ip_address="${ip_address}"
       rdt_sampling_rate="${rdt_sampling_rate}"
-      internal_filter_rate="${internal_filter_rate}"/>
+      internal_filter_rate="${internal_filter_rate}"
+      use_hardware_biasing="${use_hardware_biasing}"/>
   </xacro:macro>
 </robot>
