Commit message: works for ati sensors

File: net_ft_description/urdf/net_ft_sensor_macro.urdf.xacro (robot description, xacro)
@@ -27,4 +27,10 @@
       <xacro:property name="mesh_file" value="onrobot_hexe_v2_ft_sensor"/>
       <xacro:property name="sensor_mass" value="0.245"/>
+      <xacro:property name="sensor_radius" value="0.07"/>
+      <xacro:property name="sensor_height" value="0.0375"/>
+    </xacro:if>
+    <xacro:if value="${sensor_type == 'ati'}">
+      <xacro:property name="mesh_file" value="ati_gamma_ip65_ft_sensor"/>
+      <xacro:property name="sensor_mass" value="0.5"/>
       <xacro:property name="sensor_radius" value="0.07"/>
       <xacro:property name="sensor_height" value="0.0375"/>

Commit message: corrected the origin of the mesh files to align with the plane of the mounting side and the sensing coordinate frame, and changed naming convention for urdf macro file to clarify sensing coordinate frame

File: net_ft_description/urdf/net_ft_sensor_macro.urdf.xacro (robot description, xacro)
@@ -20,5 +20,5 @@
     </xacro:macro>
     <xacro:if value="${sensor_type == 'ati_axia'}">
-      <xacro:property name="mesh_file" value="ati_axia80_ft_sensor"/>
+      <xacro:property name="mesh_file" value="ati_axia80_ft_sensor_corrected_origin"/>
       <xacro:property name="sensor_mass" value="0.28"/>
       <xacro:property name="sensor_radius" value="0.082"/>
@@ -40,8 +40,8 @@
       <!-- The parent link must be read from the robot model it is attached to. -->
       <parent link="${parent}"/>
-      <child link="${prefix}fts_link"/>
+      <child link="${prefix}fts_base_link"/>
       <xacro:insert_block name="origin" />
     </joint>
-    <link name="${prefix}fts_link">
+    <link name="${prefix}fts_base_link">
       <visual>
         <origin xyz="0 0 0" rpy="0 0 0" />
@@ -61,9 +61,9 @@
     </link>
     <joint name="${prefix}tool_side_joint" type="fixed">
-      <parent link="${prefix}fts_link"/>
-      <child link="${prefix}tool_mount_link"/>
+      <parent link="${prefix}fts_base_link"/>
+      <child link="${prefix}sensing_link"/>
       <origin xyz="0 0 ${sensor_height}" rpy="0 0 0"/>
     </joint>
-    <link name="${prefix}tool_mount_link"/>
+    <link name="${prefix}sensing_link"/>
     <xacro:include filename="$(find net_ft_description)/urdf/net_ft_sensor.ros2_control.xacro" />
     <xacro:net_ft_sensor_ros2_control

Commit message: forgot to save the urdf file change

File: net_ft_description/urdf/net_ft_sensor_macro.urdf.xacro (robot description, xacro)
@@ -21,5 +21,5 @@
     </xacro:macro>
     <xacro:if value="${sensor_type == 'ati_axia'}">
-      <xacro:property name="mesh_file" value="ati_axia80_ft_sensor_corrected_origin"/>
+      <xacro:property name="mesh_file" value="ati_axia80_ft_sensor"/>
       <xacro:property name="sensor_mass" value="0.28"/>
       <xacro:property name="sensor_radius" value="0.082"/>
